Commit message: Added world, put arm on platform

File: urdf/ur5_with_cam.urdf.xacro (robot description, xacro)
@@ -351,36 +351,41 @@
     </joint>
     <gazebo reference="${prefix}tool0">
-      <sensor type="camera" name="camera">
-        <update_rate>30.0</update_rate>
-        <camera name="camera">
-          <horizontal_fov>1.3962634</horizontal_fov>
+      <sensor name="${prefix}tool0_camera" type="depth">
+        <update_rate>20</update_rate>
+        <camera>
+          <horizontal_fov>1.047198</horizontal_fov>
           <image>
-            <width>800</width>
-            <height>800</height>
+            <width>640</width>
+            <height>480</height>
             <format>R8G8B8</format>
           </image>
           <clip>
-            <near>0.02</near>
-            <far>300</far>
+            <near>0.05</near>
+            <far>3</far>
           </clip>
-          <noise>
-            <type>gaussian</type>
-            <mean>0.0</mean>
-            <stddev>0.007</stddev>
-          </noise>
         </camera>
-        <plugin name="camera_controller" filename="libgazebo_ros_camera.so">
+        <plugin name="${prefix}tool0_controller" filename="libgazebo_ros_openni_kinect.so">
+          <baseline>0.2</baseline>
           <alwaysOn>true</alwaysOn>
-          <updateRate>0.0</updateRate>
-          <cameraName>camera/rgb</cameraName>
-          <imageTopicName>image_raw</imageTopicName>
-          <cameraInfoTopicName>camera_info</cameraInfoTopicName>
+          <updateRate>1.0</updateRate>
+          <cameraName>camera_ir</cameraName>
+          <imageTopicName>/camera/color/image_raw</imageTopicName>
+          <cameraInfoTopicName>/camera/color/camera_info</cameraInfoTopicName>
+          <depthImageTopicName>/camera/depth/image_raw</depthImageTopicName>
+          <depthImageInfoTopicName>/camera/depth/camera_info</depthImageInfoTopicName>
+          <pointCloudTopicName>/camera/depth/points</pointCloudTopicName>
           <frameName>camera_link</frameName>
-          <hackBaseline>0.07</hackBaseline>
-          <distortionK1>0.0</distortionK1>
-          <distortionK2>0.0</distortionK2>
-          <distortionK3>0.0</distortionK3>
-          <distortionT1>0.0</distortionT1>
-          <distortionT2>0.0</distortionT2>
+          <pointCloudCutoff>0.5</pointCloudCutoff>
+          <pointCloudCutoffMax>3.0</pointCloudCutoffMax>
+          <distortionK1>0.00000001</distortionK1>
+          <distortionK2>0.00000001</distortionK2>
+          <distortionK3>0.00000001</distortionK3>
+          <distortionT1>0.00000001</distortionT1>
+          <distortionT2>0.00000001</distortionT2>
+          <CxPrime>0</CxPrime>
+          <Cx>0</Cx>
+          <Cy>0</Cy>
+          <focalLength>0</focalLength>
+          <hackBaseline>0</hackBaseline>
         </plugin>
       </sensor>

File: urdf/ur5_with_cam_robot.urdf.xacro (robot description, xacro)
@@ -11,9 +11,33 @@
     transmission_hw_interface="$(arg transmission_hw_interface)"
   />
-  <link name="world" />
+  <link name='world' />
   <joint name="world_joint" type="fixed">
     <parent link="world" />
+    <child link = "podest" />
+    <origin xyz="0.0 0.0 0.43" rpy="0.0 0.0 0.0" />
+  </joint>
+  <link name='podest'>
+    <pose>0 0 0 0 0 0</pose>
+    <inertial>
+      <mass value="1000.0"/>
+      <origin rpy="0 0 0" xyz="0 0 0"/>
+      <inertia ixx="607.975" ixy="0.0" ixz="0.0" iyy="632.875" iyz="0.0" izz="16.6"/>
+      <!-- for a box: ixx = 0.083 * mass * (y*y + z*z), ixy = 0, ixz = 0, iyy = 0.083 * mass * (x*x + z*z), iyz = 0, izz = 0.083 * mass * (x*x + y*y) -->
+    </inertial>
+    <!--collision name='collision'>
+      <geometry>
+        <box size="0.095 0.095 0.845" />
+      </geometry>
+    </collision-->
+    <visual name='visual'>
+      <geometry>
+        <box size="0.1 0.1 0.85" />
+      </geometry>
+    </visual>
+  </link>
+  <joint name="podest_joint" type="fixed">
+    <parent link="podest" />
     <child link = "base_link" />
-    <origin xyz="0.0 0.0 0.0" rpy="0.0 0.0 0.0" />
+    <origin xyz="0.0 0.0 0.43" rpy="0.0 0.0 0.0" />
   </joint>
 </robot>

Commit message: Fixed camera positioning and frames, added capsicum plant to world

File: urdf/ur5_with_cam.urdf.xacro (robot description, xacro)
@@ -350,6 +350,18 @@
       <child link="${prefix}tool0"/>
     </joint>
-    <gazebo reference="${prefix}tool0">
-      <sensor name="${prefix}tool0_camera" type="depth">
+    <link name="${prefix}camera_link"/>
+    <joint name="${prefix}tool0_camera-link_fixed_joint" type="fixed">
+      <origin xyz="0 0 0.02" rpy="0 ${pi/-2.0} ${pi/-2.0}"/>
+      <parent link="${prefix}tool0"/>
+      <child link="${prefix}camera_link"/>
+    </joint>
+    <link name="${prefix}camera_depth_frame"/>
+    <joint name="${prefix}camera-link_camera-depth_fixed_joint" type="fixed">
+      <origin xyz="0 0 0" rpy="${pi/-2.0} 0 ${pi/-2.0}"/>
+      <parent link="${prefix}camera_link"/>
+      <child link="${prefix}camera_depth_frame"/>
+    </joint>
+    <gazebo reference="${prefix}camera_link">
+      <sensor name="${prefix}camera" type="depth">
         <update_rate>20</update_rate>
         <camera>
@@ -358,5 +370,5 @@
             <width>640</width>
             <height>480</height>
-            <format>R8G8B8</format>
+            <format>B8G8R8</format>
           </image>
           <clip>
@@ -365,5 +377,5 @@
           </clip>
         </camera>
-        <plugin name="${prefix}tool0_controller" filename="libgazebo_ros_openni_kinect.so">
+        <plugin name="${prefix}camera_controller" filename="libgazebo_ros_openni_kinect.so">
           <baseline>0.2</baseline>
           <alwaysOn>true</alwaysOn>
@@ -375,5 +387,5 @@
           <depthImageInfoTopicName>/camera/depth/camera_info</depthImageInfoTopicName>
           <pointCloudTopicName>/camera/depth/points</pointCloudTopicName>
-          <frameName>camera_link</frameName>
+          <frameName>${prefix}camera_depth_frame</frameName>
           <pointCloudCutoff>0.5</pointCloudCutoff>
           <pointCloudCutoffMax>3.0</pointCloudCutoffMax>

File: urdf/ur5_with_cam_robot.urdf.xacro (robot description, xacro)
@@ -14,8 +14,8 @@
   <joint name="world_joint" type="fixed">
     <parent link="world" />
-    <child link = "podest" />
+    <child link = "platform" />
     <origin xyz="0.0 0.0 0.43" rpy="0.0 0.0 0.0" />
   </joint>
-  <link name='podest'>
+  <link name='platform'>
     <pose>0 0 0 0 0 0</pose>
     <inertial>
@@ -36,6 +36,6 @@
     </visual>
   </link>
-  <joint name="podest_joint" type="fixed">
-    <parent link="podest" />
+  <joint name="platform_joint" type="fixed">
+    <parent link="platform" />
     <child link = "base_link" />
     <origin xyz="0.0 0.0 0.43" rpy="0.0 0.0 0.0" />
