Commit message: Fixed camera_array in xacro

File: urdf/ur_with_cam.xacro (robot description, xacro)
@@ -42,7 +42,29 @@
   </xacro:if>
   <xacro:if value="${camera == 'camera_array'}">
+    <xacro:include filename="$(find ur_with_cam_gazebo)/urdf/inc/camera_array.xacro"/>
     <xacro:camera_array
       prefix=""
       parent="arm_tool0"
+      xoff="0.03"
+      yoff="0.027"
+      zoff="0.027"
+    />
+  </xacro:if>
+  <xacro:property name="camera2" value="$(arg camera2)"/>
+  <xacro:if value="${camera2 == 'depth_camera'}">
+    <xacro:include filename="$(find ur_with_cam_gazebo)/urdf/inc/depth_camera.xacro"/>
+    <xacro:depth_camera
+      prefix=""
+      parent="arm_tool0"
+    />
+  </xacro:if>
+  <xacro:if value="${camera2 == 'camera_array'}">
+    <xacro:include filename="$(find ur_with_cam_gazebo)/urdf/inc/camera_array.xacro"/>
+    <xacro:camera_array
+      prefix=""
+      parent="arm_tool0"
+      xoff="0.03"
+      yoff="0.027"
+      zoff="0.027"
     />
   </xacro:if>
