Commit message: Added collision to robot bases, limited retractable base extension to prevent collision with floor

File: urdf/inc/retractable_base.xacro (robot description, xacro)
@@ -46,4 +46,9 @@
       </geometry>
     </visual>
+    <collision>
+      <geometry>
+        <mesh filename="package://ur_with_cam_gazebo/meshes/retractable_base.dae" />
+      </geometry>
+    </collision>
     <xacro:cylinder_inertial radius="0.15" length="1.2" mass="1">
       <origin xyz="0.0 0.0 0.0" rpy="0 0 0" />
@@ -55,13 +60,18 @@
     <origin xyz="0.0 0.0 0.0" rpy="0.0 0.0 0.0" />
     <axis xyz="0 0 1" />
-    <limit lower="0" upper="1.2" effort="1000.0" velocity="3.15"/>
+    <limit lower="0" upper="0.5" effort="1000.0" velocity="3.15"/>
     <dynamics damping="0.0" friction="0.0"/>
 </joint>
 <link name="${prefix}move_z_link" >
-    <visual name='visual'>
+    <visual>
       <geometry>
         <cylinder radius="0.05" length="1.2" />
       </geometry>
     </visual>
+    <collision>
+      <geometry>
+        <cylinder radius="0.05" length="1.2" />
+      </geometry>
+    </collision>
     <xacro:cylinder_inertial radius="0.05" length="1.2" mass="1">
       <origin xyz="0.0 0.0 0.0" rpy="0 0 0" />

File: urdf/inc/static_base.xacro (robot description, xacro)
@@ -15,9 +15,14 @@
     <!-- for a box: ixx = 0.083 * mass * (y*y + z*z), ixy = 0, ixz = 0, iyy = 0.083 * mass * (x*x + z*z), iyz = 0, izz = 0.083 * mass * (x*x + y*y) -->
   </inertial>
-  <visual name='${prefix}platform_visual'>
+  <visual>
     <geometry>
-      <box size="0.1 0.1 0.85" />
+      <box size="0.1 0.1 0.82" />
     </geometry>
   </visual>
+  <collision>
+    <geometry>
+      <box size="0.1 0.1 0.82" />
+    </geometry>
+  </collision>
 </link>
 <joint name="${prefix}platform_joint" type="fixed">

Commit message: Added files to launch simulation with xarm7 (WIP)

File: urdf/inc/retractable_base.xacro (robot description, xacro)
@@ -3,5 +3,5 @@
 <xacro:include filename="$(find ur_with_cam_gazebo)/urdf/inc/retractable_base_transmissions.xacro" />
 <xacro:include filename="$(find ur_with_cam_gazebo)/urdf/inc/ur_common.xacro" />
-<xacro:macro name="retractable_base" params="prefix arm_prefix transmission_hw_interface
+<xacro:macro name="retractable_base" params="prefix arm_base_link transmission_hw_interface
     x_move_joint_lower_limit:=-1   x_move_joint_upper_limit:=1
     y_move_joint_lower_limit:=-1   y_move_joint_upper_limit:=1
@@ -78,7 +78,7 @@
     </xacro:cylinder_inertial>
 </link>
-<joint name="${prefix}${arm_prefix}base_joint" type="fixed">
+<joint name="${prefix}${arm_base_link}_joint" type="fixed">
   <parent link="${prefix}move_z_link" />
-  <child link = "${arm_prefix}base_link" />
+  <child link = "${arm_base_link}" />
   <origin xyz="0.0 0.0 0.61" rpy="0.0 0.0 0.0" />
 </joint>

File: urdf/inc/static_base.xacro (robot description, xacro)
@@ -1,5 +1,5 @@
 <?xml version="1.0"?>
 <robot name="static_base" xmlns:xacro="http://ros.org/wiki/xacro">
-<xacro:macro name="static_base" params="prefix arm_prefix">
+<xacro:macro name="static_base" params="prefix arm_base_link">
 <joint name="${prefix}world_joint" type="fixed">
   <parent link="world" />
@@ -31,9 +31,9 @@
   <origin xyz="0.0 0.0 0.43" rpy="0.0 0.0 0.0" />
 </joint>
-<xacro:if value="${arm_prefix != prefix}">
+<xacro:if value="${arm_base_link != prefix + 'base_link'}">
   <link name="${prefix}base_link" />
-  <joint name="${prefix}${arm_prefix}connection_joint" type="fixed">
+  <joint name="${prefix}${arm_base_link}_connection_joint" type="fixed">
     <parent link="${prefix}base_link" />
-    <child link = "${arm_prefix}base_link" />
+    <child link = "${arm_base_link}" />
     <origin xyz="0.0 0.0 0.0" rpy="0.0 0.0 0.0" />
   </joint>

File: urdf/inc/trolley_base.xacro (robot description, xacro)
@@ -3,5 +3,5 @@
 <xacro:include filename="$(find ur_with_cam_gazebo)/urdf/inc/trolley_base_transmissions.xacro" />
 <xacro:include filename="$(find ur_with_cam_gazebo)/urdf/inc/ur_common.xacro" />
-<xacro:macro name="trollomatic" params="prefix arm_prefix transmission_hw_interface enable_collisions:=false enable_inertia:=true">
+<xacro:macro name="trollomatic" params="prefix arm_base_link transmission_hw_interface enable_collisions:=false enable_inertia:=true">
   <xacro:property name="PI" value="3.1415926535897931"/>
   <xacro:trolley_base_transmissions prefix="${prefix}" hw_interface="${transmission_hw_interface}" />
@@ -171,8 +171,8 @@
     <link name="${prefix}tracker">
   </link>
-  <xacro:if value="${arm_prefix != prefix}">
-    <joint name="${prefix}${arm_prefix}connection_joint" type="fixed">
+  <xacro:if value="${arm_base_link != prefix + 'base_link'}">
+    <joint name="${prefix}${arm_base_link}_connection_joint" type="fixed">
       <parent link="${prefix}platform_base" />
-      <child link = "${arm_prefix}base_link" />
+      <child link = "${arm_base_link}" />
       <origin xyz="0.49 0.03 0.1" rpy="0.0 0.0 0.0" />
     </joint>

File: urdf/ur_with_cam.xacro (robot description, xacro)
@@ -1,10 +1,8 @@
 <?xml version="1.0"?>
 <robot xmlns:xacro="http://wiki.ros.org/xacro" name="ur_with_cam" >
-  <xacro:include filename="$(find ur_with_cam_gazebo)/urdf/inc/ur_gazebo.xacro"/>
-  <!--Declare arguments -->
-  <xacro:arg name="joint_limit_params" default=""/>
-  <xacro:arg name="physical_params" default=""/>
-  <xacro:arg name="kinematics_params" default=""/>
-  <xacro:arg name="visual_params" default=""/>
+  <xacro:arg name="arm" default="ur5e"/>
+  <xacro:arg name="base" default="static"/>
+  <xacro:arg name="camera" default="depth_camera"/>
+  <xacro:arg name="camera2" default=""/>
   <!--
     legal values:
@@ -16,21 +14,64 @@
   -->
   <xacro:arg name="transmission_hw_interface" default="hardware_interface/PositionJointInterface"/>
-  <xacro:arg name="safety_limits" default="false"/>
-  <xacro:arg name="safety_pos_margin" default="0.15"/>
-  <xacro:arg name="safety_k_position" default="20"/>
-  <xacro:arg name="base" default="static"/>
-  <xacro:arg name="camera" default="depth_camera"/>
-  <xacro:arg name="camera2" default=""/>
-  <xacro:ur_robot_gazebo
-    prefix="arm_"
-    joint_limits_parameters_file="$(arg joint_limit_params)"
-    kinematics_parameters_file="$(arg kinematics_params)"
-    physical_parameters_file="$(arg physical_params)"
-    visual_parameters_file="$(arg visual_params)"
-    transmission_hw_interface="$(arg transmission_hw_interface)"
-    safety_limits="$(arg safety_limits)"
-    safety_pos_margin="$(arg safety_pos_margin)"
-    safety_k_position="$(arg safety_k_position)"
-  />
+  <xacro:property name="arm" value="$(arg arm)"/>
+  <xacro:if value="${arm == 'ur5e'}">
+    <xacro:include filename="$(find ur_with_cam_gazebo)/urdf/inc/ur_gazebo.xacro"/>
+    <!--Declare arguments -->
+    <xacro:arg name="joint_limit_params" default=""/>
+    <xacro:arg name="physical_params" default=""/>
+    <xacro:arg name="kinematics_params" default=""/>
+    <xacro:arg name="visual_params" default=""/>
+    <xacro:arg name="safety_limits" default="false"/>
+    <xacro:arg name="safety_pos_margin" default="0.15"/>
+    <xacro:arg name="safety_k_position" default="20"/>
+    <xacro:ur_robot_gazebo
+      prefix="arm_"
+      joint_limits_parameters_file="$(arg joint_limit_params)"
+      kinematics_parameters_file="$(arg kinematics_params)"
+      physical_parameters_file="$(arg physical_params)"
+      visual_parameters_file="$(arg visual_params)"
+      transmission_hw_interface="$(arg transmission_hw_interface)"
+      safety_limits="$(arg safety_limits)"
+      safety_pos_margin="$(arg safety_pos_margin)"
+      safety_k_position="$(arg safety_k_position)"
+    />
+    <!-- ${prefix}base_link -> ${prefix}tool0-->
+    <xacro:property name="arm_base_link" value="arm_base_link"/>
+    <xacro:property name="tool_link" value="arm_tool0"/>
+  </xacro:if>
+  <xacro:if value="${arm == 'xarm7'}">
+    <xacro:arg name="prefix" default=""/>
+    <xacro:arg name="ros_namespace" default="xarm"/>
+    <xacro:arg name="limited" default="false"/>
+    <xacro:arg name="effort_control" default="false"/>
+    <xacro:arg name="velocity_control" default="false"/>
+    <xacro:arg name="add_other_geometry" default="false"/>
+    <xacro:arg name="geometry_type" default="box"/>
+    <xacro:arg name="geometry_mass" default="0.1"/>
+    <xacro:arg name="geometry_height" default="0.1"/>
+    <xacro:arg name="geometry_radius" default="0.1"/>
+    <xacro:arg name="geometry_length" default="0.1"/>
+    <xacro:arg name="geometry_width" default="0.1"/>
+    <xacro:arg name="geometry_mesh_filename" default=""/>
+    <xacro:arg name="geometry_mesh_origin_xyz" default="0 0 0"/>
+    <xacro:arg name="geometry_mesh_origin_rpy" default="0 0 0"/>
+    <xacro:arg name="geometry_mesh_tcp_xyz" default="0 0 0"/>
+    <xacro:arg name="geometry_mesh_tcp_rpy" default="0 0 0"/>
+    <!-- load xarm7 robot -->
+    <xacro:include filename="$(find ur_with_cam_gazebo)/urdf/inc/xarm7_robot_macro.xacro" />
+    <xacro:xarm7_robot prefix="$(arg prefix)" namespace="$(arg ros_namespace)" limited="$(arg limited)"
+      effort_control="$(arg effort_control)" velocity_control="$(arg velocity_control)"
+      add_other_geometry="$(arg add_other_geometry)"
+      geometry_type="$(arg geometry_type)" geometry_mass="$(arg geometry_mass)"
+      geometry_height="$(arg geometry_height)" geometry_radius="$(arg geometry_radius)"
+      geometry_length="$(arg geometry_length)" geometry_width="$(arg geometry_width)"
+      geometry_mesh_filename="$(arg geometry_mesh_filename)"
+      geometry_mesh_origin_xyz="$(arg geometry_mesh_origin_xyz)" geometry_mesh_origin_rpy="$(arg geometry_mesh_origin_rpy)"
+      geometry_mesh_tcp_xyz="$(arg geometry_mesh_tcp_xyz)" geometry_mesh_tcp_rpy="$(arg geometry_mesh_tcp_rpy)"
+    />
+    <!--${prefix}link_base -> ${prefix}link_eef -->
+    <xacro:property name="arm_base_link" value="link_base"/>
+    <xacro:property name="tool_link" value="link_eef"/>
+  </xacro:if>
   <xacro:property name="camera" value="$(arg camera)"/>
   <xacro:if value="${camera == 'depth_camera'}">
@@ -38,5 +79,5 @@
     <xacro:depth_camera
       prefix=""
-      parent="arm_tool0"
+      parent="${tool_link}"
     />
   </xacro:if>
@@ -45,5 +86,5 @@
     <xacro:camera_array
       prefix=""
-      parent="arm_tool0"
+      parent="${tool_link}"
       xoff="0.03"
       yoff="0.027"
@@ -55,5 +96,5 @@
     <xacro:l515
       prefix=""
-      parent="arm_tool0"
+      parent="${tool_link}"
       use_nominal_extrinsics="false"
     />
@@ -63,5 +104,5 @@
     <xacro:d435
       prefix=""
-      parent="arm_tool0"
+      parent="${tool_link}"
       use_nominal_extrinsics="false"
     />
@@ -72,5 +113,5 @@
     <xacro:depth_camera
       prefix=""
-      parent="arm_tool0"
+      parent="${tool_link}"
     />
   </xacro:if>
@@ -79,5 +120,5 @@
     <xacro:camera_array
       prefix=""
-      parent="arm_tool0"
+      parent="${tool_link}"
       xoff="0.03"
       yoff="0.027"
@@ -91,5 +132,5 @@
     <xacro:static_base
       prefix=""
-      arm_prefix="arm_"
+      arm_base_link="${arm_base_link}"
     />
   </xacro:if>
@@ -98,5 +139,5 @@
     <xacro:retractable_base
       prefix=""
-      arm_prefix="arm_"
+      arm_base_link="${arm_base_link}"
       transmission_hw_interface="$(arg transmission_hw_interface)"
     />
@@ -106,5 +147,5 @@
     <xacro:trollomatic
       prefix=""
-      arm_prefix="arm_"
+      arm_base_link="${arm_base_link}"
       transmission_hw_interface="$(arg transmission_hw_interface)"
     />
