Commit message: Add rail base initial joint values, add floor to urdf to prevent collision

File: urdf/inc/rail_base.xacro (robot description, xacro)
@@ -1,4 +1,4 @@
 <?xml version="1.0"?>
-<robot name="retractable_base" xmlns:xacro="http://ros.org/wiki/xacro">
+<robot name="rail_base" xmlns:xacro="http://ros.org/wiki/xacro">
 <xacro:include filename="$(find ur_with_cam_gazebo)/urdf/inc/rail_base_transmissions.xacro" />
 <xacro:include filename="$(find ur_with_cam_gazebo)/urdf/inc/ur_common.xacro" />

File: urdf/ur_with_cam.xacro (robot description, xacro)
@@ -22,4 +22,5 @@
   <xacro:arg name="camera" default="depth_camera"/>
   <xacro:arg name="camera2" default=""/>
+  <xacro:arg name="include_room" default="true"/>
   <xacro:ur_robot_gazebo
     prefix="arm_"
@@ -118,3 +119,8 @@
     />
   </xacro:if>
+  <xacro:property name="include_room" value="$(arg include_room)"/>
+  <xacro:if value="${include_room}">
+    <xacro:include filename="$(find ur_with_cam_gazebo)/urdf/inc/room.xacro"/>
+    <xacro:room/>
+  </xacro:if>
 </robot>
