Commit message: updated trolley based on phenorob_ur5e trolley configuration

File: urdf/inc/trolley_base.xacro (robot description, xacro)
@@ -119,4 +119,21 @@
     </xacro:if>
   </link>
+  <link name="${prefix}platform_base_arm">
+    <visual>
+      <geometry>
+          <mesh filename="package://ur_with_cam_gazebo/meshes/arm_base_platform.dae" />
+        <!-- For inertia computation, see: http://gazebosim.org/tutorials?tut=inertia&cat=build_robot-->
+      </geometry>
+    </visual>
+    <xacro:if value="${enable_collisions}">
+      <collision>
+        <geometry>
+            <!-- <mesh filename="package://ur_with_cam_gazebo/meshes/arm_base_platform_with_corridor.dae" /> -->
+            <mesh filename="package://ur_with_cam_gazebo/meshes/arm_base_platform.dae" />
+          <!-- For inertia computation, see: http://gazebosim.org/tutorials?tut=inertia&cat=build_robot-->
+        </geometry>
+      </collision>
+    </xacro:if>
+  </link>
   <!--joint name="platform_base_to_control_box" type="fixed">
     <origin xyz="1.19 0 0.04" rpy="0 0 0"/>
@@ -135,4 +152,9 @@
     </visual>
   </link-->
+  <joint name="arm_base_arm_joint" type="fixed">
+    <parent link="${prefix}platform_base" />
+    <child link = "${prefix}platform_base_arm" />
+    <origin xyz="0 0 0" rpy="0.0 0.0 0.0" />
+  </joint>
   <!-- Camera fixed joints -->
   <joint name="${prefix}base_link_to_cam0" type="fixed">
@@ -175,5 +197,5 @@
       <parent link="${prefix}platform_base" />
       <child link = "${arm_prefix}base_link" />
-      <origin xyz="0.49 0.03 0.1" rpy="0.0 0.0 0.0" />
+      <origin xyz="0.1 -0.11 0.1" rpy="0.0 0.0 0.0" />
     </joint>
   </xacro:if>

Commit message: enabled collisions for trolley and fixed the shaking issue. but inertias may need modifications

File: urdf/inc/trolley_base.xacro (robot description, xacro)
@@ -3,5 +3,5 @@
 <xacro:include filename="$(find ur_with_cam_gazebo)/urdf/inc/trolley_base_transmissions.xacro" />
 <xacro:include filename="$(find ur_with_cam_gazebo)/urdf/inc/ur_common.xacro" />
-<xacro:macro name="trollomatic" params="prefix arm_prefix transmission_hw_interface enable_collisions:=false enable_inertia:=true">
+<xacro:macro name="trollomatic" params="prefix arm_prefix transmission_hw_interface enable_collisions:=true enable_inertia:=true">
   <xacro:property name="PI" value="3.1415926535897931"/>
   <xacro:trolley_base_transmissions prefix="${prefix}" hw_interface="${transmission_hw_interface}" />
@@ -15,7 +15,18 @@
   </joint>
   <link name="${prefix}platform_start_link">
+    <!--
     <xacro:cylinder_inertial radius="0.06" length="0.2" mass="1">
       <origin xyz="0.0 0.0 0.0" rpy="0 0 0" />
     </xacro:cylinder_inertial>
+    -->
+    <!-- TODO: TEMPORARY FIX -->
+      <inertial>
+        <mass value="1.0"/>
+        <origin rpy="0 0 0" xyz="0 0 0"/>
+      <inertia
+        ixx="0.1" ixy="0.0" ixz="0.0"
+        iyy="0.1" iyz="0.0"
+        izz="0.1"/>
+      </inertial>
   </link>
   <joint name="${prefix}platform_move_joint" type="prismatic">
@@ -136,4 +147,45 @@
     </xacro:if>
   </link>
+  <!-- for decreasing shaking -->
+  <gazebo reference="${prefix}platform_base">
+    <kp>1000000.0</kp>
+    <kd>1.0</kd>
+    <mu1>0.8</mu1>
+    <mu2>0.8</mu2>
+    <maxVel>0.0</maxVel>
+    <minDepth>0.001</minDepth>
+  </gazebo>
+  <gazebo reference="${prefix}platform_base_arm">
+    <kp>1000000.0</kp>
+    <kd>1.0</kd>
+    <mu1>0.8</mu1>
+    <mu2>0.8</mu2>
+    <maxVel>0.0</maxVel>
+    <minDepth>0.001</minDepth>
+  </gazebo>
+  <gazebo reference="${prefix}platform_lift_joint">
+    <kp>1000000.0</kp>
+    <kd>1.0</kd>
+    <mu1>0.8</mu1>
+    <mu2>0.8</mu2>
+    <maxVel>0.0</maxVel>
+    <minDepth>0.001</minDepth>
+  </gazebo>
+  <gazebo reference="${prefix}base_link">
+    <kp>1000000.0</kp>
+    <kd>1.0</kd>
+    <mu1>0.8</mu1>
+    <mu2>0.8</mu2>
+    <maxVel>0.0</maxVel>
+    <minDepth>0.001</minDepth>
+  </gazebo>
+  <gazebo reference="${prefix}platform_start_link">
+    <kp>1000000.0</kp>
+    <kd>1.0</kd>
+    <mu1>0.8</mu1>
+    <mu2>0.8</mu2>
+    <maxVel>0.0</maxVel>
+    <minDepth>0.001</minDepth>
+  </gazebo>
   <!--joint name="platform_base_to_control_box" type="fixed">
     <origin xyz="1.19 0 0.04" rpy="0 0 0"/>

Commit message: added cart_nopipe.stl model. set as the default model for trolley.

File: urdf/inc/trolley_base.xacro (robot description, xacro)
@@ -41,5 +41,6 @@
     <visual>
         <geometry>
-            <mesh filename="package://ur_with_cam_gazebo/meshes/cart.stl" scale="0.001 0.001 0.001"/>
+            <!--<mesh filename="package://ur_with_cam_gazebo/meshes/cart.stl" scale="0.001 0.001 0.001"/>-->
+            <mesh filename="package://ur_with_cam_gazebo/meshes/cart_nopipe.stl" scale="0.001 0.001 0.001"/>
             <!-- For inertia computation, see: http://gazebosim.org/tutorials?tut=inertia&cat=build_robot
             Mesh Bounding Box Size 2.022500 0.778000 2.816000
@@ -67,5 +68,6 @@
       <collision>
         <geometry>
-          <mesh filename="package://ur_with_cam_gazebo/meshes/cart.stl" scale="0.001 0.001 0.001"/>
+          <!--<mesh filename="package://ur_with_cam_gazebo/meshes/cart.stl" scale="0.001 0.001 0.001"/>-->
+          <mesh filename="package://ur_with_cam_gazebo/meshes/cart_nopipe.stl" scale="0.001 0.001 0.001"/>
         </geometry>
         <origin xyz="0 0 0" rpy="0 0 ${PI}"/>

Commit message: Change trolley orientation to work with world22

File: urdf/inc/trolley_base.xacro (robot description, xacro)
@@ -12,5 +12,5 @@
     <parent link="world" />
     <child link = "${prefix}platform_start_link" />
-    <origin xyz="-2.0 0.0 0.12" rpy="0.0 0.0 0.0" />
+    <origin xyz="0.0 0.0 0.12" rpy="0.0 0.0 ${pi/2}" />
   </joint>
   <link name="${prefix}platform_start_link">
@@ -31,5 +31,5 @@
   </link>
   <joint name="${prefix}platform_move_joint" type="prismatic">
-    <origin xyz="0.0 0.0 0.0" rpy="0.0 0.0 0.0" />
+    <origin xyz="-2.0 0.0 0.0" rpy="0.0 0.0 0.0" />
     <axis xyz="1 0 0"/>
     <limit upper="4.0" lower="0.0" effort="1000" velocity="1.0"/>

Commit message: Adjust launch for simulated trolley
- additional pose_frame parameter
- home_flipped pose in srdf
- adjust workspacce
- adjust maximum move length of trolley

File: urdf/inc/trolley_base.xacro (robot description, xacro)
@@ -33,5 +33,5 @@
     <origin xyz="-2.0 0.0 0.0" rpy="0.0 0.0 0.0" />
     <axis xyz="1 0 0"/>
-    <limit upper="4.0" lower="0.0" effort="1000" velocity="1.0"/>
+    <limit upper="3.0" lower="0.0" effort="1000" velocity="1.0"/>
     <parent link="${prefix}platform_start_link" />
     <child link = "${prefix}base_link" />
